Commit message: feat: enhance Curobo V2 IK solver with waist yaw constraints
- Updated the Curobo V2 IK solver to include waist yaw limits, enhancing stability during inverse kinematics calculations.
- Modified the IK configuration to enforce constraints on waist pitch and yaw, ensuring more accurate joint positioning.
- Added support for compiled costs in the planning module, allowing for efficient cost management.
- Adjusted URDF files to correct joint axis orientations and improve collision detection.
- Enhanced documentation to reflect new constraints and configuration options.

File: autolife_planning/resources/robot/autolife/autolife.urdf (robot description, URDF)
Before this commit: robot autolife, 44 links, 43 joints
Joints:
- joint Joint_Left_Wrist_Upper: axis 0 0 1 -> 0 0 -1

File: autolife_planning/resources/robot/autolife/autolife_base.urdf (robot description, URDF)
Before this commit: robot autolife, 47 links, 46 joints
Joints:
- joint Joint_Left_Wrist_Upper: axis 0 0 1 -> 0 0 -1

File: autolife_planning/resources/robot/autolife/autolife_base_simple.urdf (robot description, URDF)
Before this commit: robot autolife, 38 links, 37 joints
Joints:
- joint Joint_Left_Wrist_Upper: axis 0 0 1 -> 0 0 -1

File: autolife_planning/resources/robot/autolife/autolife_simple.urdf (robot description, URDF)
Before this commit: robot autolife, 35 links, 34 joints
Joints:
- joint Joint_Left_Wrist_Upper: axis 0 0 1 -> 0 0 -1

File: autolife_planning/resources/robot/autolife/autolife_spherized.urdf (robot description, URDF)
Before this commit: robot autolife, 38 links, 37 joints
Links:
- link Link_Ankle_to_Knee: geometry collision sphere radius=0.051865; collision sphere radius=0.064405
- link Link_Knee_to_Waist_Pitch: geometry collision sphere radius=0.05; collision sphere radius=0.05
- link Link_Left_Gripper: geometry collision sphere radius=0.014861; collision sphere radius=0.014924
- link Link_Left_Gripper_Left_Inner_Knuckle: geometry collision sphere radius=0.007688; collision sphere radius=0.008259
- link Link_Left_Gripper_Right_Inner_Knuckle: geometry collision sphere radius=0.007758; collision sphere radius=0.007785
- link Link_Left_Gripper_Right_Outer_Knuckle: geometry collision sphere radius=0.013022; collision sphere radius=0.01446
- link Link_Left_UpperArm_to_Elbow: geometry collision sphere radius=0.047211; collision sphere radius=0.049776
- link Link_Left_Wrist_Lower_to_Gripper: geometry collision sphere radius=0.025046; collision sphere radius=0.027008
- link Link_Neck_Pitch_to_Neck_Yaw: geometry collision sphere radius=0.019273; collision sphere radius=0.021156
- link Link_Right_Gripper: geometry collision sphere radius=0.011516; collision sphere radius=0.013694
- link Link_Right_Gripper_Left_Inner_Knuckle: geometry collision sphere radius=0.006091; collision sphere radius=0.006866
- link Link_Right_Gripper_Right_Inner_Knuckle: geometry collision sphere radius=0.006983; collision sphere radius=0.007098
- link Link_Right_Gripper_Right_Outer_Knuckle: geometry collision sphere radius=0.013137; collision sphere radius=0.014168
- link Link_Right_UpperArm_to_Elbow: geometry collision sphere radius=0.049052; collision sphere radius=0.050831
- link Link_Right_Wrist_Lower_to_Gripper: geometry collision sphere radius=0.022846; collision sphere radius=0.02285
- link Link_Waist_Yaw_to_Shoulder_Inner: geometry collision sphere radius=0.087293; collision sphere radius=0.116
Joints:
- joint Joint_Left_Wrist_Upper: axis 0 0 1 -> 0 0 -1

File: autolife_planning/resources/robot/autolife/autolife_viz.urdf (robot description, URDF)
Before this commit: robot autolife, 44 links, 43 joints
Joints:
- joint Joint_Left_Gripper_Left_Finger: mimic (none) -> joint=Joint_Left_Gripper multiplier=-1 offset=0
- joint Joint_Left_Gripper_Left_Inner_Knuckle: mimic (none) -> joint=Joint_Left_Gripper multiplier=1 offset=0
- joint Joint_Left_Gripper_Right_Finger: mimic (none) -> joint=Joint_Left_Gripper multiplier=1 offset=0
- joint Joint_Left_Gripper_Right_Inner_Knuckle: mimic (none) -> joint=Joint_Left_Gripper multiplier=-1 offset=0
- joint Joint_Left_Gripper_Right_Outer_Knuckle: mimic (none) -> joint=Joint_Left_Gripper multiplier=-1 offset=0
- joint Joint_Left_Wrist_Upper: axis 0 0 1 -> 0 0 -1
- joint Joint_Right_Gripper_Left_Finger: mimic (none) -> joint=Joint_Right_Gripper multiplier=-1 offset=0
- joint Joint_Right_Gripper_Left_Inner_Knuckle: mimic (none) -> joint=Joint_Right_Gripper multiplier=1 offset=0
- joint Joint_Right_Gripper_Right_Finger: mimic (none) -> joint=Joint_Right_Gripper multiplier=1 offset=0
- joint Joint_Right_Gripper_Right_Inner_Knuckle: mimic (none) -> joint=Joint_Right_Gripper multiplier=-1 offset=0
- joint Joint_Right_Gripper_Right_Outer_Knuckle: mimic (none) -> joint=Joint_Right_Gripper multiplier=-1 offset=0
