Commit message: Overleaf Connect auto-sync [2026-09-29 12:05:23]

File: resources/robot/autolife/autolife_spherized.urdf (robot description, URDF)
Before this commit: robot autolife, 39 links, 38 joints
Links:
- link Link_Ankle_to_Knee: geometry collision sphere radius=0.097339; collision sphere radius=0.100443
- link Link_Ground_Vehicle: geometry collision sphere radius=0.228216; collision sphere radius=0.229268
- link Link_Head: geometry collision sphere radius=0.104034; collision sphere radius=0.107025
- link Link_Knee_to_Waist_Pitch: geometry collision sphere radius=0.133092; collision sphere radius=0.141159
- link Link_Left_Elbow_to_Forearm: geometry collision sphere radius=0.072483; collision sphere radius=0.074207
- link Link_Left_Forearm_to_Wrist_Upper: geometry collision sphere radius=0.063514; collision sphere radius=0.063956
- link Link_Left_Gripper: geometry collision sphere radius=0.010772; collision sphere radius=0.015258
- link Link_Left_Gripper_Left_Finger: geometry collision sphere radius=0.012766; collision sphere radius=0.01407
- link Link_Left_Gripper_Left_Inner_Knuckle: geometry collision sphere radius=0.01108; collision sphere radius=0.011429
- link Link_Left_Gripper_Right_Finger: geometry collision sphere radius=0.013132; collision sphere radius=0.013205
- link Link_Left_Gripper_Right_Inner_Knuckle: geometry collision sphere radius=0.010106; collision sphere radius=0.013005
- link Link_Left_Gripper_Right_Outer_Knuckle: geometry collision sphere radius=0.018138; collision sphere radius=0.020794
- link Link_Left_Shoulder_Inner_to_Shoulder_Outer: geometry collision sphere radius=0.07272; collision sphere radius=0.075542
- link Link_Left_Shoulder_Outer_to_UpperArm: geometry collision sphere radius=0.049416; collision sphere radius=0.052103
- link Link_Left_UpperArm_to_Elbow: geometry collision sphere radius=0.064875; collision sphere radius=0.068368
- link Link_Left_Wrist_Lower_to_Gripper: geometry collision sphere radius=0.026463; collision sphere radius=0.032636
- link Link_Left_Wrist_Upper_to_Wrist_Lower: geometry collision sphere radius=0.060718; collision sphere radius=0.06172
- link Link_Neck_Pitch_to_Neck_Yaw: geometry collision sphere radius=0.020382; collision sphere radius=0.020783
- link Link_Neck_Roll_to_Neck_Pitch: geometry collision sphere radius=0.033579; collision sphere radius=0.034495
- link Link_Neck_Yaw_to_Head: geometry collision sphere radius=0.046122; visual mesh filename=package://meshes/Link_Neck_Yaw_to_Head.STL
- link Link_Right_Elbow_to_Forearm: geometry collision sphere radius=0.066045; collision sphere radius=0.067801
- link Link_Right_Forearm_to_Wrist_Upper: geometry collision sphere radius=0.063533; collision sphere radius=0.064658
- link Link_Right_Gripper: geometry collision sphere radius=0.012907; collision sphere radius=0.013993
- link Link_Right_Gripper_Left_Finger: geometry collision sphere radius=0.011624; collision sphere radius=0.013743
- link Link_Right_Gripper_Left_Inner_Knuckle: geometry collision sphere radius=0.010216; collision sphere radius=0.011139
- link Link_Right_Gripper_Right_Finger: geometry collision sphere radius=0.011515; collision sphere radius=0.016205
- link Link_Right_Gripper_Right_Inner_Knuckle: geometry collision sphere radius=0.010299; collision sphere radius=0.011137
- link Link_Right_Gripper_Right_Outer_Knuckle: geometry collision sphere radius=0.012618; collision sphere radius=0.01268
- link Link_Right_Shoulder_Inner_to_Shoulder_Outer: geometry collision sphere radius=0.072711; collision sphere radius=0.074985
- link Link_Right_Shoulder_Outer_to_UpperArm: geometry collision sphere radius=0.048692; collision sphere radius=0.049497
- link Link_Right_UpperArm_to_Elbow: geometry collision sphere radius=0.063863; collision sphere radius=0.070081
- link Link_Right_Wrist_Lower_to_Gripper: geometry collision sphere radius=0.024127; collision sphere radius=0.026286
- link Link_Right_Wrist_Upper_to_Wrist_Lower: geometry collision sphere radius=0.061351; collision sphere radius=0.061609
- link Link_Waist_Pitch_to_Waist_Yaw: geometry collision sphere radius=0.095622; collision sphere radius=0.095822
- link Link_Waist_Yaw_to_Shoulder_Inner: geometry collision sphere radius=0.166372; collision sphere radius=0.188175

Commit message: Revert "Overleaf Connect auto-sync [2026-09-29 12:05:23]"
This reverts commit 3b7febb4fd051e4ae69678b04121bf2a054bb5aa.

An Overleaf Connect auto-sync committed an in-progress working tree
directly to main, together with LaTeX/Overleaf .gitignore entries and
local submodule checkouts.  Restore main to 53848b3; the intended
changes come in through a pull request.

File: resources/robot/autolife/autolife_spherized.urdf (robot description, URDF)
Before this commit: robot autolife, 39 links, 38 joints
Links:
- link Link_Ankle_to_Knee: geometry collision sphere radius=0.065401; collision sphere radius=0.083369
- link Link_Ground_Vehicle: geometry collision sphere radius=0.124736; collision sphere radius=0.134366
- link Link_Head: geometry collision sphere radius=0.058381; collision sphere radius=0.077592
- link Link_Knee_to_Waist_Pitch: geometry collision sphere radius=0.060682; collision sphere radius=0.061545
- link Link_Left_Elbow_to_Forearm: geometry collision sphere radius=0.047232; collision sphere radius=0.047431
- link Link_Left_Forearm_to_Wrist_Upper: geometry collision sphere radius=0.040536; collision sphere radius=0.049415
- link Link_Left_Gripper: geometry collision sphere radius=0.006469; collision sphere radius=0.009258
- link Link_Left_Gripper_Left_Finger: geometry collision sphere radius=0.006321; collision sphere radius=0.00773
- link Link_Left_Gripper_Left_Inner_Knuckle: geometry collision sphere radius=0.008167; collision sphere radius=0.008891
- link Link_Left_Gripper_Right_Finger: geometry collision sphere radius=0.00615; collision sphere radius=0.007988
- link Link_Left_Gripper_Right_Inner_Knuckle: geometry collision sphere radius=0.008923; collision sphere radius=0.00908
- link Link_Left_Gripper_Right_Outer_Knuckle: geometry collision sphere radius=0.009322; collision sphere radius=0.00942
- link Link_Left_Shoulder_Inner_to_Shoulder_Outer: geometry collision sphere radius=0.013394; collision sphere radius=0.014002
- link Link_Left_Shoulder_Outer_to_UpperArm: geometry collision sphere radius=0.00672; collision sphere radius=0.009657
- link Link_Left_UpperArm_to_Elbow: geometry collision sphere radius=0.03254; collision sphere radius=0.037461
- link Link_Left_Wrist_Lower_to_Gripper: geometry collision sphere radius=0.022696; collision sphere radius=0.022829
- link Link_Left_Wrist_Upper_to_Wrist_Lower: geometry collision sphere radius=0.032954; collision sphere radius=0.04234
- link Link_Neck_Pitch_to_Neck_Yaw: geometry collision sphere radius=0.030683; collision sphere radius=0.031251
- link Link_Neck_Roll_to_Neck_Pitch: geometry collision sphere radius=0.020922; collision sphere radius=0.022565
- link Link_Neck_Yaw_to_Head: geometry collision sphere radius=0.024508; collision sphere radius=0.024842
- link Link_Right_Elbow_to_Forearm: geometry collision sphere radius=0.038106; collision sphere radius=0.038674
- link Link_Right_Forearm_to_Wrist_Upper: geometry collision sphere radius=0.047294; collision sphere radius=0.048996
- link Link_Right_Gripper: geometry collision sphere radius=0.008755; collision sphere radius=0.010239
- link Link_Right_Gripper_Left_Finger: geometry collision sphere radius=0.007344; collision sphere radius=0.008111
- link Link_Right_Gripper_Left_Inner_Knuckle: geometry collision sphere radius=0.010125; collision sphere radius=0.010413
- link Link_Right_Gripper_Right_Finger: geometry collision sphere radius=0.007741; collision sphere radius=0.008174
- link Link_Right_Gripper_Right_Inner_Knuckle: geometry collision sphere radius=0.010724; collision sphere radius=0.01078
- link Link_Right_Gripper_Right_Outer_Knuckle: geometry collision sphere radius=0.009767; collision sphere radius=0.010619
- link Link_Right_Shoulder_Inner_to_Shoulder_Outer: geometry collision sphere radius=0.017547; collision sphere radius=0.018656
- link Link_Right_Shoulder_Outer_to_UpperArm: geometry collision sphere radius=0.009632; collision sphere radius=0.01072
- link Link_Right_UpperArm_to_Elbow: geometry collision sphere radius=0.034332; collision sphere radius=0.035037
- link Link_Right_Wrist_Lower_to_Gripper: geometry collision sphere radius=0.022929; collision sphere radius=0.024794
- link Link_Right_Wrist_Upper_to_Wrist_Lower: geometry collision sphere radius=0.032954; collision sphere radius=0.04234
- link Link_Waist_Pitch_to_Waist_Yaw: geometry collision sphere radius=0.05068; collision sphere radius=0.064037
- link Link_Waist_Yaw_to_Shoulder_Inner: geometry collision sphere radius=0.029842; collision sphere radius=0.032967
